File: Hardware/PCB-aux/waveshaper-aux/waveshaperxy.kicad_pcb (KiCad board)
At the start: 2 copper layers, 189 x 174 mm, 63 parts, among them J1 2x7 IDC header, J10 AudioJack2_SwitchT, J11 2_pin_Molex_header, J12 AudioJack2_SwitchT, J13 3_pin_Molex_header, J14 2x5 pin socket, J15 AudioJack2_SwitchT, J16 AudioJack2_SwitchT, J17 AudioJack2_SwitchT, J18 AudioJack2_SwitchT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

Commit message: Use TL074
Parts:
- U3, U4: value TL074 -> MCP6004
Routing:
- net +12V: track 232.2 -> 214.0 mm, vias 0 -> 3
- net Net-(J9-Pad5): track 127.4 -> 145.0 mm, vias 0 -> 1
- net MIXIN_+1: track 42.9 -> 60.3 mm
- net Net-(J9-Pad3): track 173.7 -> 188.5 mm, vias 0 -> 1
- net MIXIN_0: track 45.2 -> 59.4 mm, vias 0 -> 3
- net Net-(J9-Pad4): track 140.6 -> 129.7 mm, vias 0 -> 1
- net -12V: track 43.7 -> 54.5 mm
- net /RIPOUT_0: track 33.0 -> 42.9 mm, vias 0 -> 1
- net /Panel and power/+12V_IN: track 11.1 -> 20.5 mm
- net P_-2: track 42.8 -> 51.2 mm, vias 0 -> 2
- net Net-(J9-Pad7): track 86.8 -> 94.8 mm, vias 0 -> 1
- net P_-1: track 71.7 -> 79.6 mm, vias 0 -> 1
- net /RIPOUT_-3: track 27.7 -> 35.2 mm, vias 0 -> 1
- net Net-(J9-Pad9): track 47.5 -> 53.7 mm
- net MIXIN_+2: track 34.0 -> 40.0 mm, vias 0 -> 1
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